File: pcb/multi_fpga/layout.kicad_pcb (KiCad board)
At the start: 2 copper layers, 479.3 x 629.7 mm, 199 parts, among them U1 Comment, U10 Comment, U11 Comment, U12 Comment, U13 Comment, U14 Comment, U15 Comment, U16 Comment, U17 Comment, U18 Comment, U19 Comment, U2 Comment, U20 Comment, U21 Comment, U22 Comment, U23 Comment, U24 Comment, U25 Comment, U26 Comment, U27 Comment, U28 Comment, U29 Comment, U3 Comment, U30 Comment, U31 Comment, U32 Comment, U33 Comment, U34 Comment, U35 Comment, U36 Comment, U37 Comment, U38 Comment, U39 Comment, U4 Comment, U40 Comment, U41 Comment, U42 Comment, U43 Comment, U44 Comment, U45 Comment, U46 Comment, U47 Comment, U48 Comment, U49 Comment, U5 Comment, U50 Comment, U51 Comment, U52 Comment, U53 Comment, U54 Comment, U55 Comment, U56 Comment, U57 Comment, U58 Comment, U59 Comment, U6 Comment, U60 Comment, U61 Comment, U62 Comment, U63 Comment, U64 Comment, U65 Comment, U66 Comment, U67 Comment, U68 Comment, U69 Comment, U7 Comment, U70 Comment, U71 Comment, U72 Comment, U73 Comment, U74 Comment, U75 Comment, U76 Comment, U77 Comment, U78 Comment, U79 Comment, U8 Comment, U80 Comment, U81 Comment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

Commit message: Moved FPGA.
Parts:
- moved A1 117.8 mm to (46.6, 156.2), turned to 16.5985 degrees
- moved A2 117.8 mm to (-156.2, 46.6), turned to -73.4015 degrees
- moved A3 117.8 mm to (-46.6, -156.2), turned to -163.401 degrees
- moved A4 117.8 mm to (156.2, -46.6), turned to 106.599 degrees
- moved A5 9.36 mm to (-70.0, -335.6)
- moved A6 9.36 mm to (18.0, -335.6)
- moved Y1 9.36 mm to (50.0, -335.6)
Other:
- board size 479.3 x 629.7 mm -> 460.6 x 611 mm

Commit message: Changed to place cmod s7 modules radially.
Parts:
- moved A1 119.2 mm to (34.6, 37.6), turned to 51.224 degrees
- moved A2 119.2 mm to (-37.6, 34.6), turned to -38.776 degrees
- moved A3 119.2 mm to (-34.6, -37.6), turned to -128.776 degrees
- moved A4 119.2 mm to (37.6, -34.6), turned to 141.224 degrees
- moved A5 75.6 mm to (-70.0, -260.0)
- moved A6 75.6 mm to (18.0, -260.0)
- moved Y1 75.6 mm to (50.0, -260.0)
Other:
- board size 460.6 x 611 mm -> 309.6 x 459.8 mm

Commit message: Adjusted location of cmod S7 modules.
Parts:
- moved A1 36.9 mm to (56.2, 67.5), turned to 30 degrees
- moved A2 36.9 mm to (-67.5, 56.2), turned to -60 degrees
- moved A3 36.9 mm to (-56.2, -67.5), turned to -150 degrees
- moved A4 36.9 mm to (67.5, -56.2), turned to 120 degrees

Commit message: Updated with b-2-b connectors.
Parts:
- added H1A, H1B: MountingHole_2.7mm_M2.5, MountingHole_2.7mm_M2.5, F.Cu at (34.7, 79.9)
- added H1E1: MountingHole_3.2mm_M3, MountingHole_3.2mm_M3, F.Cu at (121.4, 69.7)
- added H1E2: MountingHole_3.2mm_M3, MountingHole_3.2mm_M3, F.Cu at (-47.6, 131.7)
- added H2A, H2B: MountingHole_2.7mm_M2.5, MountingHole_2.7mm_M2.5, F.Cu at (-79.9, 34.7)
- added H2E1: MountingHole_3.2mm_M3, MountingHole_3.2mm_M3, F.Cu at (-69.7, 121.4)
- added H2E2: MountingHole_3.2mm_M3, MountingHole_3.2mm_M3, F.Cu at (-131.7, -47.6)
- added H3A, H3B: MountingHole_2.7mm_M2.5, MountingHole_2.7mm_M2.5, F.Cu at (-34.7, -79.9)
- added H3E1: MountingHole_3.2mm_M3, MountingHole_3.2mm_M3, F.Cu at (-121.4, -69.7)
- added H3E2: MountingHole_3.2mm_M3, MountingHole_3.2mm_M3, F.Cu at (47.6, -131.7)
- added H4A, H4B: MountingHole_2.7mm_M2.5, MountingHole_2.7mm_M2.5, F.Cu at (79.9, -34.7)
- added H4E1: MountingHole_3.2mm_M3, MountingHole_3.2mm_M3, F.Cu at (69.7, -121.4)
- added H4E2: MountingHole_3.2mm_M3, MountingHole_3.2mm_M3, F.Cu at (131.7, 47.6)
- added HCAM1: MountingHole_2.7mm_M2.5, MountingHole_2.7mm_M2.5, F.Cu at (-10.5, 0.00)
- added HCAM2: MountingHole_2.7mm_M2.5, MountingHole_2.7mm_M2.5, F.Cu at (10.5, 0.00)
- added HPI1: MountingHole_2.7mm_M2.5, MountingHole_2.7mm_M2.5, F.Cu at (-29.0, -184.5)
- added HPI2: MountingHole_2.7mm_M2.5, MountingHole_2.7mm_M2.5, F.Cu at (29.0, -184.5)
- added HPI3: MountingHole_2.7mm_M2.5, MountingHole_2.7mm_M2.5, F.Cu at (-29.0, -135.5)
- added HPI4: MountingHole_2.7mm_M2.5, MountingHole_2.7mm_M2.5, F.Cu at (29.0, -135.5)
- added J1: PinSocket_2x06_P2.54mm_Vertical, PinSocket_2x06_P2.54mm_Vertical, F.Cu at (56.2, 67.5)
- added J2: PinSocket_2x06_P2.54mm_Vertical, PinSocket_2x06_P2.54mm_Vertical, F.Cu at (-67.5, 56.2)
- added J3: PinSocket_2x06_P2.54mm_Vertical, PinSocket_2x06_P2.54mm_Vertical, F.Cu at (-56.2, -67.5)
- added J4: PinSocket_2x06_P2.54mm_Vertical, PinSocket_2x06_P2.54mm_Vertical, F.Cu at (67.5, -56.2)
- moved A5 352.9 mm to (-7.96, 87.4), turned to -5.2 degrees
- moved A6 267.2 mm to (-64.7, -5.89), turned to -95.2 degrees
- moved Y1 200.2 mm to (5.89, -64.7)
Other:
- board size 309.6 x 459.8 mm -> 309.6 x 309.6 mm
