File: pcb/multi_fpga/arm_00.kicad_sch (KiCad schematic)
At the start: 16 parts, among them U1 IM72D128V01XTMA1, U2 IM72D128V01XTMA1, U3 IM72D128V01XTMA1, U4 IM72D128V01XTMA1, U5 IM72D128V01XTMA1, U6 IM72D128V01XTMA1, U7 IM72D128V01XTMA1, U8 IM72D128V01XTMA1

Commit message: Fixed library and power issues.
Parts:
- C1, C2, C3, C4, C5, C6, C7, C8: symbol C -> multi_fpga:C
- U1, U2, U3, U4, U5, U6, U7, U8: symbol IM72D128 -> multi_fpga:IM72D128
Changed lines of the file:
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@@
 	)
 	(symbol
-		(lib_id "C")
+		(lib_id "multi_fpga:C")
 		(at 261.62 58.42 0)
 		(unit 1)
@@
 	)
 	(symbol
-		(lib_id "C")
+		(lib_id "multi_fpga:C")
 		(at 106.68 95.25 0)
 		(unit 1)
@@
 	)
 	(symbol
-		(lib_id "IM72D128")
+		(lib_id "multi_fpga:IM72D128")
 		(at 252.73 184.15 0)
 		(unit 1)
@@
 	)
 	(symbol
-		(lib_id "power:C0_1V8")
+		(lib_id "multi_fpga:C0_1V8")
 		(at 252.73 90.17 0)
 		(unit 1)
@@
 	)
 	(symbol
-		(lib_id "IM72D128")
+		(lib_id "multi_fpga:IM72D128")
 		(at 102.87 223.52 0)
 		(unit 1)
@@
 	)
 	(symbol
-		(lib_id "C")
+		(lib_id "multi_fpga:C")
 		(at 260.35 171.45 0)
 		(unit 1)
@@
 	)
 	(symbol
-		(lib_id "C")
+		(lib_id "multi_fpga:C")
 		(at 256.54 95.25 0)
 		(unit 1)
@@
 	)
 	(symbol
-		(lib_id "IM72D128")
+		(lib_id "multi_fpga:IM72D128")
 		(at 252.73 223.52 0)
 		(unit 1)
@@
 	)
 	(symbol
-		(lib_id "IM72D128")
+		(lib_id "multi_fpga:IM72D128")
 		(at 102.87 69.85 0)
 		(unit 1)
@@
 	)
 	(symbol
-		(lib_id "power:C0_1V8")
+		(lib_id "multi_fpga:C0_1V8")
 		(at 95.25 222.25 0)
 		(unit 1)
@@
 	)
 	(symbol
-		(lib_id "power:C0_1V8")
+		(lib_id "multi_fpga:C0_1V8")
 		(at 102.87 88.9 0)
 		(unit 1)
@@
 	)
 	(symbol
-		(lib_id "C")
+		(lib_id "multi_fpga:C")
 		(at 107.95 210.82 0)
 		(unit 1)
@@
 	)
 	(symbol
-		(lib_id "power:C0_1V8")
+		(lib_id "multi_fpga:C0_1V8")
 		(at 252.73 203.2 0)
 		(unit 1)
@@
 	)
 	(symbol
-		(lib_id "power:C0_1V8")
+		(lib_id "multi_fpga:C0_1V8")
 		(at 252.73 52.07 0)
 		(unit 1)
@@
 	)
 	(symbol
-		(lib_id "C")
+		(lib_id "multi_fpga:C")
 		(at 257.81 212.09 0)
 		(unit 1)
@@
 	)
 	(symbol
-		(lib_id "power:C0_1V8")
+		(lib_id "multi_fpga:C0_1V8")
 		(at 243.84 222.25 0)
 		(unit 1)
@@
 	)
 	(symbol
-		(lib_id "IM72D128")
+		(lib_id "multi_fpga:IM72D128")
 		(at 102.87 184.15 0)
 		(unit 1)
@@
 	)
 	(symbol
-		(lib_id "IM72D128")
+		(lib_id "multi_fpga:IM72D128")
 		(at 102.87 109.22 0)
 		(unit 1)
@@
 	)
 	(symbol
-		(lib_id "power:C0_1V8")
+		(lib_id "multi_fpga:C0_1V8")
 		(at 102.87 53.34 0)
 		(unit 1)
@@
 	)
 	(symbol
-		(lib_id "C")
+		(lib_id "multi_fpga:C")
 		(at 109.22 170.18 0)
 		(unit 1)
@@
 	)
 	(symbol
-		(lib_id "power:C0_1V8")
+		(lib_id "multi_fpga:C0_1V8")
 		(at 102.87 163.83 0)
 		(unit 1)
@@
 	)
 	(symbol
-		(lib_id "power:C0_1V8")
+		(lib_id "multi_fpga:C0_1V8")
 		(at 102.87 203.2 0)
 		(unit 1)
@@
 	)
 	(symbol
-		(lib_id "IM72D128")
+		(lib_id "multi_fpga:IM72D128")
 		(at 252.73 69.85 0)
 		(unit 1)
@@
 	)
 	(symbol
-		(lib_id "power:C0_1V8")
+		(lib_id "multi_fpga:C0_1V8")
 		(at 243.84 107.95 0)
 		(unit 1)
@@
 	)
 	(symbol
-		(lib_id "power:C0_1V8")
+		(lib_id "multi_fpga:C0_1V8")
 		(at 93.98 107.95 0)
 		(unit 1)
@@
 	)
 	(symbol
-		(lib_id "power:C0_1V8")
+		(lib_id "multi_fpga:C0_1V8")
 		(at 252.73 162.56 0)
 		(unit 1)
@@
 	)
 	(symbol
-		(lib_id "C")
+		(lib_id "multi_fpga:C")
 		(at 111.76 58.42 0)
 		(unit 1)
@@
 	)
 	(symbol
-		(lib_id "IM72D128")
+		(lib_id "multi_fpga:IM72D128")
 		(at 252.73 109.22 0)
 		(unit 1)

Commit message: Fixed power and C ref des collisions.
Parts:
- renumbered C2 to C1, C4 to C2, C1 to C4, C6 to C5, C8 to C6, C5 to C8

Commit message: Fixed C and PWR ref des errors.
Parts:
- renumbered C4 to C1, C1 to C2, C2 to C4, C8 to C5, C5 to C6, C6 to C8
Changed lines of the file:
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@@
 		(in_pos_files yes)
 		(dnp no)
-		(property "Reference" "#PWR019"
+		(property "Reference" "#PWR0033"
 			(at 243.84 182.88 0)
 			(hide yes)
@@
 		(in_pos_files yes)
 		(dnp no)
-		(property "Reference" "C8"
+		(property "Reference" "C5"
 			(at 263.62 56.92 0)
 			(show_name no)
@@
 		(in_pos_files yes)
 		(dnp no)
-		(property "Reference" "#PWR022"
+		(property "Reference" "#PWR0022"
 			(at 252.73 76.2 0)
 			(hide yes)
@@
 		(in_pos_files yes)
 		(dnp no)
-		(property "Reference" "C1"
+		(property "Reference" "C2"
 			(at 108.68 93.75 0)
 			(show_name no)
@@
 		(in_pos_files yes)
 		(dnp no)
-		(property "Reference" "#PWR013"
+		(property "Reference" "#PWR0010"
 			(at 106.68 99.06 0)
 			(hide yes)
@@
 		(in_pos_files yes)
 		(dnp no)
-		(property "Reference" "#PWR030"
+		(property "Reference" "#PWR0040"
 			(at 257.81 215.9 0)
 			(hide yes)
@@
 		(in_pos_files yes)
 		(dnp no)
-		(property "Reference" "#PWR014"
+		(property "Reference" "#PWR0020"
 			(at 107.95 214.63 0)
 			(hide yes)
@@
 		(in_pos_files yes)
 		(dnp no)
-		(property "Reference" "#PWR016"
+		(property "Reference" "#PWR0005"
 			(at 111.76 62.23 0)
 			(hide yes)
@@
 		(in_pos_files yes)
 		(dnp no)
-		(property "Reference" "#PWR023"
+		(property "Reference" "#PWR0026"
 			(at 252.73 90.17 0)
 			(hide yes)
@@
 		(in_pos_files yes)
 		(dnp no)
-		(property "Reference" "#PWR032"
+		(property "Reference" "#PWR0025"
 			(at 261.62 62.23 0)
 			(hide yes)
@@
 		(in_pos_files yes)
 		(dnp no)
-		(property "Reference" "C5"
+		(property "Reference" "C6"
 			(at 258.54 93.75 0)
 			(show_name no)
@@
 		(in_pos_files yes)
 		(dnp no)
-		(property "Reference" "#PWR028"
+		(property "Reference" "#PWR0037"
 			(at 252.73 229.87 0)
 			(hide yes)
@@
 		(in_pos_files yes)
 		(dnp no)
-		(property "Reference" "#PWR08"
+		(property "Reference" "#PWR0007"
 			(at 102.87 115.57 0)
 			(hide yes)
@@
 		(in_pos_files yes)
 		(dnp no)
-		(property "Reference" "#PWR029"
+		(property "Reference" "#PWR0030"
 			(at 256.54 99.06 0)
 			(hide yes)
@@
 		(in_pos_files yes)
 		(dnp no)
-		(property "Reference" "#PWR01"
+		(property "Reference" "#PWR0003"
 			(at 93.98 68.58 0)
 			(hide yes)
@@
 		(in_pos_files yes)
 		(dnp no)
-		(property "Reference" "#PWR026"
+		(property "Reference" "#PWR0032"
 			(at 252.73 190.5 0)
 			(hide yes)
@@
 		(in_pos_files yes)
 		(dnp no)
-		(property "Reference" "#PWR04"
+		(property "Reference" "#PWR0018"
 			(at 95.25 222.25 0)
 			(hide yes)
@@
 		(in_pos_files yes)
 		(dnp no)
-		(property "Reference" "#PWR031"
+		(property "Reference" "#PWR0035"
 			(at 260.35 175.26 0)
 			(hide yes)
@@
 		(in_pos_files yes)
 		(dnp no)
-		(property "Reference" "#PWR07"
+		(property "Reference" "#PWR0006"
 			(at 102.87 88.9 0)
 			(hide yes)
@@
 		(in_pos_files yes)
 		(dnp no)
-		(property "Reference" "#PWR017"
+		(property "Reference" "#PWR0023"
 			(at 243.84 68.58 0)
 			(hide yes)
@@
 		(in_pos_files yes)
 		(dnp no)
-		(property "Reference" "C2"
+		(property "Reference" "C4"
 			(at 109.95 209.32 0)
 			(show_name no)
@@
 		(in_pos_files yes)
 		(dnp no)
-		(property "Reference" "#PWR06"
+		(property "Reference" "#PWR0002"
 			(at 102.87 76.2 0)
 			(hide yes)
@@
 		(in_pos_files yes)
 		(dnp no)
-		(property "Reference" "#PWR027"
+		(property "Reference" "#PWR0036"
 			(at 252.73 203.2 0)
 			(hide yes)
@@
 		(in_pos_files yes)
 		(dnp no)
-		(property "Reference" "#PWR021"
+		(property "Reference" "#PWR0021"
 			(at 252.73 52.07 0)
 			(hide yes)
@@
 		(in_pos_files yes)
 		(dnp no)
-		(property "Reference" "C6"
+		(property "Reference" "C8"
 			(at 259.81 210.59 0)
 			(show_name no)
@@
 		(in_pos_files yes)
 		(dnp no)
-		(property "Reference" "#PWR020"
+		(property "Reference" "#PWR0038"
 			(at 243.84 222.25 0)
 			(hide yes)
@@
 		(in_pos_files yes)
 		(dnp no)
-		(property "Reference" "#PWR05"
+		(property "Reference" "#PWR0001"
 			(at 102.87 53.34 0)
 			(hide yes)
@@
 		(in_pos_files yes)
 		(dnp no)
-		(property "Reference" "#PWR09"
+		(property "Reference" "#PWR0011"
 			(at 102.87 163.83 0)
 			(hide yes)
@@
 		(in_pos_files yes)
 		(dnp no)
-		(property "Reference" "#PWR011"
+		(property "Reference" "#PWR0016"
 			(at 102.87 203.2 0)
 			(hide yes)
@@
 		(in_pos_files yes)
 		(dnp no)
-		(property "Reference" "#PWR018"
+		(property "Reference" "#PWR0028"
 			(at 243.84 107.95 0)
 			(hide yes)
@@
 		(in_pos_files yes)
 		(dnp no)
-		(property "Reference" "#PWR010"
+		(property "Reference" "#PWR0012"
 			(at 102.87 190.5 0)
 			(hide yes)
@@
 		(in_pos_files yes)
 		(dnp no)
-		(property "Reference" "#PWR02"
+		(property "Reference" "#PWR0008"
 			(at 93.98 107.95 0)
 			(hide yes)
@@
 		(in_pos_files yes)
 		(dnp no)
-		(property "Reference" "#PWR025"
+		(property "Reference" "#PWR0031"
 			(at 252.73 162.56 0)
 			(hide yes)
@@
 		(in_pos_files yes)
 		(dnp no)
-		(property "Reference" "C4"
+		(property "Reference" "C1"
 			(at 113.76 56.92 0)
 			(show_name no)
@@
 		(in_pos_files yes)
 		(dnp no)
-		(property "Reference" "#PWR012"
+		(property "Reference" "#PWR0017"
 			(at 102.87 229.87 0)
 			(hide yes)
@@
 		(in_pos_files yes)
 		(dnp no)
-		(property "Reference" "#PWR03"
+		(property "Reference" "#PWR0013"
 			(at 93.98 182.88 0)
 			(hide yes)
@@
 		(in_pos_files yes)
 		(dnp no)
-		(property "Reference" "#PWR024"
+		(property "Reference" "#PWR0027"
 			(at 252.73 115.57 0)
 			(hide yes)
@@
 		(in_pos_files yes)
 		(dnp no)
-		(property "Reference" "#PWR015"
+		(property "Reference" "#PWR0015"
 			(at 109.22 173.99 0)
 			(hide yes)
@@
 		)
 	)
-	(embedded_fonts no)
 )

Commit message: Global fix of res defs.
Parts:
- renumbered C2 to C18, C4 to C19, C3 to C20, C1 to C21, C6 to C22, C8 to C23, C7 to C24, C5 to C25

Commit message: Changed to use generic cap symbols and footprints.
Parts:
- C18, C19, C20, C21, C22, C23, C24, C25: footprint (none) -> Capacitor_SMD:C_0603_1608Metric; symbol multi_fpga:C -> Device:C
Changed lines of the file:
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@@
 	)
 	(symbol
-		(lib_id "multi_fpga:C")
+		(lib_id "Device:C")
 		(at 261.62 58.42 0)
 		(unit 1)
@@
 			)
 		)
-		(property "Footprint" ""
-			(at 261.62 58.42 0)
+		(property "Footprint" "Capacitor_SMD:C_0603_1608Metric"
+			(at 262.5852 62.23 0)
 			(hide yes)
 			(show_name no)
@@
 			)
 		)
-		(property "Description" "100 nF decoupling capacitor, 0402"
+		(property "Description" "Unpolarized capacitor"
 			(at 261.62 58.42 0)
 			(hide yes)
@@
 	)
 	(symbol
-		(lib_id "multi_fpga:C")
+		(lib_id "Device:C")
 		(at 106.68 95.25 0)
 		(unit 1)
@@
 			)
 		)
-		(property "Footprint" ""
-			(at 106.68 95.25 0)
+		(property "Footprint" "Capacitor_SMD:C_0603_1608Metric"
+			(at 107.6452 99.06 0)
 			(hide yes)
 			(show_name no)
@@
 			)
 		)
-		(property "Description" "100 nF decoupling capacitor, 0402"
+		(property "Description" "Unpolarized capacitor"
 			(at 106.68 95.25 0)
 			(hide yes)
@@
 	)
 	(symbol
-		(lib_id "multi_fpga:C")
+		(lib_id "Device:C")
 		(at 260.35 171.45 0)
 		(unit 1)
@@
 			)
 		)
-		(property "Footprint" ""
-			(at 260.35 171.45 0)
+		(property "Footprint" "Capacitor_SMD:C_0603_1608Metric"
+			(at 261.3152 175.26 0)
 			(hide yes)
 			(show_name no)
@@
 			)
 		)
-		(property "Description" "100 nF decoupling capacitor, 0402"
+		(property "Description" "Unpolarized capacitor"
 			(at 260.35 171.45 0)
 			(hide yes)
@@
 	)
 	(symbol
-		(lib_id "multi_fpga:C")
+		(lib_id "Device:C")
 		(at 256.54 95.25 0)
 		(unit 1)
@@
 			)
 		)
-		(property "Footprint" ""
-			(at 256.54 95.25 0)
+		(property "Footprint" "Capacitor_SMD:C_0603_1608Metric"
+			(at 257.5052 99.06 0)
 			(hide yes)
 			(show_name no)
@@
 			)
 		)
-		(property "Description" "100 nF decoupling capacitor, 0402"
+		(property "Description" "Unpolarized capacitor"
 			(at 256.54 95.25 0)
 			(hide yes)
@@
 	)
 	(symbol
-		(lib_id "multi_fpga:C")
+		(lib_id "Device:C")
 		(at 107.95 210.82 0)
 		(unit 1)
@@
 			)
 		)
-		(property "Footprint" ""
-			(at 107.95 210.82 0)
+		(property "Footprint" "Capacitor_SMD:C_0603_1608Metric"
+			(at 108.9152 214.63 0)
 			(hide yes)
 			(show_name no)
@@
 			)
 		)
-		(property "Description" "100 nF decoupling capacitor, 0402"
+		(property "Description" "Unpolarized capacitor"
 			(at 107.95 210.82 0)
 			(hide yes)
@@
 	)
 	(symbol
-		(lib_id "multi_fpga:C")
+		(lib_id "Device:C")
 		(at 257.81 212.09 0)
 		(unit 1)
@@
 			)
 		)
-		(property "Footprint" ""
-			(at 257.81 212.09 0)
+		(property "Footprint" "Capacitor_SMD:C_0603_1608Metric"
+			(at 258.7752 215.9 0)
 			(hide yes)
 			(show_name no)
@@
 			)
 		)
-		(property "Description" "100 nF decoupling capacitor, 0402"
+		(property "Description" "Unpolarized capacitor"
 			(at 257.81 212.09 0)
 			(hide yes)
@@
 	)
 	(symbol
-		(lib_id "multi_fpga:C")
+		(lib_id "Device:C")
 		(at 109.22 170.18 0)
 		(unit 1)
@@
 			)
 		)
-		(property "Footprint" ""
-			(at 109.22 170.18 0)
+		(property "Footprint" "Capacitor_SMD:C_0603_1608Metric"
+			(at 110.1852 173.99 0)
 			(hide yes)
 			(show_name no)
@@
 			)
 		)
-		(property "Description" "100 nF decoupling capacitor, 0402"
+		(property "Description" "Unpolarized capacitor"
 			(at 109.22 170.18 0)
 			(hide yes)
@@
 	)
 	(symbol
-		(lib_id "multi_fpga:C")
+		(lib_id "Device:C")
 		(at 111.76 58.42 0)
 		(unit 1)
@@
 			)
 		)
-		(property "Footprint" ""
-			(at 111.76 58.42 0)
+		(property "Footprint" "Capacitor_SMD:C_0603_1608Metric"
+			(at 112.7252 62.23 0)
 			(hide yes)
 			(show_name no)
@@
 			)
 		)
-		(property "Description" "100 nF decoupling capacitor, 0402"
+		(property "Description" "Unpolarized capacitor"
 			(at 111.76 58.42 0)
 			(hide yes)
