File: pcb/multi_fpga/arm_05.kicad_sch (KiCad schematic)
At the start: 16 parts, among them U41 IM72D128V01XTMA1, U42 IM72D128V01XTMA1, U43 IM72D128V01XTMA1, U44 IM72D128V01XTMA1, U45 IM72D128V01XTMA1, U46 IM72D128V01XTMA1, U47 IM72D128V01XTMA1, U48 IM72D128V01XTMA1

Commit message: Changed to use generic cap symbols and footprints.
Parts:
- C58, C59, C60, C61, C62, C63, C64, C65: symbol multi_fpga:C -> Device:C
Changed lines of the file:
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@@
 	)
 	(symbol
-		(lib_id "multi_fpga:C")
+		(lib_id "Device:C")
 		(at 261.62 58.42 0)
 		(unit 1)
@@
 		)
 		(property "Footprint" ""
-			(at 261.62 58.42 0)
+			(at 262.5852 62.23 0)
 			(hide yes)
 			(show_name no)
@@
 			)
 		)
-		(property "Description" "100 nF decoupling capacitor, 0402"
+		(property "Description" "Unpolarized capacitor"
 			(at 261.62 58.42 0)
 			(hide yes)
@@
 	)
 	(symbol
-		(lib_id "multi_fpga:C")
+		(lib_id "Device:C")
 		(at 260.35 171.45 0)
 		(unit 1)
@@
 		)
 		(property "Footprint" ""
-			(at 260.35 171.45 0)
+			(at 261.3152 175.26 0)
 			(hide yes)
 			(show_name no)
@@
 			)
 		)
-		(property "Description" "100 nF decoupling capacitor, 0402"
+		(property "Description" "Unpolarized capacitor"
 			(at 260.35 171.45 0)
 			(hide yes)
@@
 	)
 	(symbol
-		(lib_id "multi_fpga:C")
+		(lib_id "Device:C")
 		(at 107.95 210.82 0)
 		(unit 1)
@@
 		)
 		(property "Footprint" ""
-			(at 107.95 210.82 0)
+			(at 108.9152 214.63 0)
 			(hide yes)
 			(show_name no)
@@
 			)
 		)
-		(property "Description" "100 nF decoupling capacitor, 0402"
+		(property "Description" "Unpolarized capacitor"
 			(at 107.95 210.82 0)
 			(hide yes)
@@
 	)
 	(symbol
-		(lib_id "multi_fpga:C")
+		(lib_id "Device:C")
 		(at 256.54 95.25 0)
 		(unit 1)
@@
 		)
 		(property "Footprint" ""
-			(at 256.54 95.25 0)
+			(at 257.5052 99.06 0)
 			(hide yes)
 			(show_name no)
@@
 			)
 		)
-		(property "Description" "100 nF decoupling capacitor, 0402"
+		(property "Description" "Unpolarized capacitor"
 			(at 256.54 95.25 0)
 			(hide yes)
@@
 	)
 	(symbol
-		(lib_id "multi_fpga:C")
+		(lib_id "Device:C")
 		(at 109.22 170.18 0)
 		(unit 1)
@@
 		)
 		(property "Footprint" ""
-			(at 109.22 170.18 0)
+			(at 110.1852 173.99 0)
 			(hide yes)
 			(show_name no)
@@
 			)
 		)
-		(property "Description" "100 nF decoupling capacitor, 0402"
+		(property "Description" "Unpolarized capacitor"
 			(at 109.22 170.18 0)
 			(hide yes)
@@
 	)
 	(symbol
-		(lib_id "multi_fpga:C")
+		(lib_id "Device:C")
 		(at 111.76 58.42 0)
 		(unit 1)
@@
 		)
 		(property "Footprint" ""
-			(at 111.76 58.42 0)
+			(at 112.7252 62.23 0)
 			(hide yes)
 			(show_name no)
@@
 			)
 		)
-		(property "Description" "100 nF decoupling capacitor, 0402"
+		(property "Description" "Unpolarized capacitor"
 			(at 111.76 58.42 0)
 			(hide yes)
@@
 	)
 	(symbol
-		(lib_id "multi_fpga:C")
+		(lib_id "Device:C")
 		(at 106.68 95.25 0)
 		(unit 1)
@@
 		)
 		(property "Footprint" ""
-			(at 106.68 95.25 0)
+			(at 107.6452 99.06 0)
 			(hide yes)
 			(show_name no)
@@
 			)
 		)
-		(property "Description" "100 nF decoupling capacitor, 0402"
+		(property "Description" "Unpolarized capacitor"
 			(at 106.68 95.25 0)
 			(hide yes)
@@
 	)
 	(symbol
-		(lib_id "multi_fpga:C")
+		(lib_id "Device:C")
 		(at 257.81 212.09 0)
 		(unit 1)
@@
 		)
 		(property "Footprint" ""
-			(at 257.81 212.09 0)
+			(at 258.7752 215.9 0)
 			(hide yes)
 			(show_name no)
@@
 			)
 		)
-		(property "Description" "100 nF decoupling capacitor, 0402"
+		(property "Description" "Unpolarized capacitor"
 			(at 257.81 212.09 0)
 			(hide yes)

Commit message: Added stock footprints for C symbols.
Parts:
- C58, C59, C60, C61, C62, C63, C64, C65: footprint (none) -> Capacitor_SMD:C_0603_1608Metric
Changed lines of the file:
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@@
 			)
 		)
-		(property "Footprint" ""
+		(property "Footprint" "Capacitor_SMD:C_0603_1608Metric"
 			(at 262.5852 62.23 0)
 			(hide yes)
@@
 			)
 		)
-		(property "Footprint" ""
+		(property "Footprint" "Capacitor_SMD:C_0603_1608Metric"
 			(at 261.3152 175.26 0)
 			(hide yes)
@@
 			)
 		)
-		(property "Footprint" ""
+		(property "Footprint" "Capacitor_SMD:C_0603_1608Metric"
 			(at 108.9152 214.63 0)
 			(hide yes)
@@
 			)
 		)
-		(property "Footprint" ""
+		(property "Footprint" "Capacitor_SMD:C_0603_1608Metric"
 			(at 257.5052 99.06 0)
 			(hide yes)
@@
 			)
 		)
-		(property "Footprint" ""
+		(property "Footprint" "Capacitor_SMD:C_0603_1608Metric"
 			(at 110.1852 173.99 0)
 			(hide yes)
@@
 			)
 		)
-		(property "Footprint" ""
+		(property "Footprint" "Capacitor_SMD:C_0603_1608Metric"
 			(at 112.7252 62.23 0)
 			(hide yes)
@@
 			)
 		)
-		(property "Footprint" ""
+		(property "Footprint" "Capacitor_SMD:C_0603_1608Metric"
 			(at 107.6452 99.06 0)
 			(hide yes)
@@
 			)
 		)
-		(property "Footprint" ""
+		(property "Footprint" "Capacitor_SMD:C_0603_1608Metric"
 			(at 258.7752 215.9 0)
 			(hide yes)
