File: pcb/multi_fpga/arm_10.kicad_sch (KiCad schematic)
At the start: 16 parts, among them U81 IM72D128V01XTMA1, U82 IM72D128V01XTMA1, U83 IM72D128V01XTMA1, U84 IM72D128V01XTMA1, U85 IM72D128V01XTMA1, U86 IM72D128V01XTMA1, U87 IM72D128V01XTMA1, U88 IM72D128V01XTMA1

Commit message: Global fix of res defs.
Parts:
- renumbered C85 to C100, C83 to C101, C87 to C102, C88 to C103, C82 to C104, C81 to C105, C86 to C98, C84 to C99, U86 to U81, U84 to U82, U82 to U83, U87 to U84, U83 to U85, U88 to U86, U81 to U87, U85 to U88

Commit message: Changed to use generic cap symbols and footprints.
Parts:
- C100, C101, C102, C103, C104, C105, C98, C99: symbol multi_fpga:C -> Device:C
Changed lines of the file:
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@@
 	)
 	(symbol
-		(lib_id "multi_fpga:C")
+		(lib_id "Device:C")
 		(at 106.68 95.25 0)
 		(unit 1)
@@
 		)
 		(property "Footprint" ""
+			(at 107.6452 99.06 0)
+			(hide yes)
+			(show_name no)
+			(do_not_autoplace no)
+			(effects
+				(font
+					(size 1.27 1.27)
+				)
+			)
+		)
+		(property "Datasheet" ""
 			(at 106.68 95.25 0)
 			(hide yes)
@@
 			)
 		)
-		(property "Datasheet" ""
+		(property "Description" "Unpolarized capacitor"
 			(at 106.68 95.25 0)
 			(hide yes)
@@
 			)
 		)
-		(property "Description" "100 nF decoupling capacitor, 0402"
-			(at 106.68 95.25 0)
-			(hide yes)
-			(show_name no)
-			(do_not_autoplace no)
-			(effects
-				(font
-					(size 1.27 1.27)
-				)
-			)
-		)
 		(pin "1"
 		)
@@
 	)
 	(symbol
-		(lib_id "multi_fpga:C")
+		(lib_id "Device:C")
 		(at 257.81 212.09 0)
 		(unit 1)
@@
 		)
 		(property "Footprint" ""
+			(at 258.7752 215.9 0)
+			(hide yes)
+			(show_name no)
+			(do_not_autoplace no)
+			(effects
+				(font
+					(size 1.27 1.27)
+				)
+			)
+		)
+		(property "Datasheet" ""
 			(at 257.81 212.09 0)
 			(hide yes)
@@
 			)
 		)
-		(property "Datasheet" ""
-			(at 257.81 212.09 0)
-			(hide yes)
-			(show_name no)
-			(do_not_autoplace no)
-			(effects
-				(font
-					(size 1.27 1.27)
-				)
-			)
-		)
-		(property "Description" "100 nF decoupling capacitor, 0402"
+		(property "Description" "Unpolarized capacitor"
 			(at 257.81 212.09 0)
 			(hide yes)
@@
 	)
 	(symbol
-		(lib_id "multi_fpga:C")
+		(lib_id "Device:C")
 		(at 107.95 210.82 0)
 		(unit 1)
@@
 		)
 		(property "Footprint" ""
+			(at 108.9152 214.63 0)
+			(hide yes)
+			(show_name no)
+			(do_not_autoplace no)
+			(effects
+				(font
+					(size 1.27 1.27)
+				)
+			)
+		)
+		(property "Datasheet" ""
 			(at 107.95 210.82 0)
 			(hide yes)
@@
 			)
 		)
-		(property "Datasheet" ""
-			(at 107.95 210.82 0)
-			(hide yes)
-			(show_name no)
-			(do_not_autoplace no)
-			(effects
-				(font
-					(size 1.27 1.27)
-				)
-			)
-		)
-		(property "Description" "100 nF decoupling capacitor, 0402"
+		(property "Description" "Unpolarized capacitor"
 			(at 107.95 210.82 0)
 			(hide yes)
@@
 	)
 	(symbol
-		(lib_id "multi_fpga:C")
+		(lib_id "Device:C")
 		(at 261.62 58.42 0)
 		(unit 1)
@@
 		)
 		(property "Footprint" ""
+			(at 262.5852 62.23 0)
+			(hide yes)
+			(show_name no)
+			(do_not_autoplace no)
+			(effects
+				(font
+					(size 1.27 1.27)
+				)
+			)
+		)
+		(property "Datasheet" ""
 			(at 261.62 58.42 0)
 			(hide yes)
@@
 			)
 		)
-		(property "Datasheet" ""
-			(at 261.62 58.42 0)
-			(hide yes)
-			(show_name no)
-			(do_not_autoplace no)
-			(effects
-				(font
-					(size 1.27 1.27)
-				)
-			)
-		)
-		(property "Description" "100 nF decoupling capacitor, 0402"
+		(property "Description" "Unpolarized capacitor"
 			(at 261.62 58.42 0)
 			(hide yes)
@@
 	)
 	(symbol
-		(lib_id "multi_fpga:C")
+		(lib_id "Device:C")
 		(at 256.54 95.25 0)
 		(unit 1)
@@
 		)
 		(property "Footprint" ""
+			(at 257.5052 99.06 0)
+			(hide yes)
+			(show_name no)
+			(do_not_autoplace no)
+			(effects
+				(font
+					(size 1.27 1.27)
+				)
+			)
+		)
+		(property "Datasheet" ""
 			(at 256.54 95.25 0)
 			(hide yes)
@@
 			)
 		)
-		(property "Datasheet" ""
+		(property "Description" "Unpolarized capacitor"
 			(at 256.54 95.25 0)
 			(hide yes)
@@
 			)
 		)
-		(property "Description" "100 nF decoupling capacitor, 0402"
-			(at 256.54 95.25 0)
-			(hide yes)
-			(show_name no)
-			(do_not_autoplace no)
-			(effects
-				(font
-					(size 1.27 1.27)
-				)
-			)
-		)
 		(pin "1"
 		)
@@
 	)
 	(symbol
-		(lib_id "multi_fpga:C")
+		(lib_id "Device:C")
 		(at 260.35 171.45 0)
 		(unit 1)
@@
 		)
 		(property "Footprint" ""
+			(at 261.3152 175.26 0)
+			(hide yes)
+			(show_name no)
+			(do_not_autoplace no)
+			(effects
+				(font
+					(size 1.27 1.27)
+				)
+			)
+		)
+		(property "Datasheet" ""
 			(at 260.35 171.45 0)
 			(hide yes)
@@
 			)
 		)
-		(property "Datasheet" ""
-			(at 260.35 171.45 0)
-			(hide yes)
-			(show_name no)
-			(do_not_autoplace no)
-			(effects
-				(font
-					(size 1.27 1.27)
-				)
-			)
-		)
-		(property "Description" "100 nF decoupling capacitor, 0402"
+		(property "Description" "Unpolarized capacitor"
 			(at 260.35 171.45 0)
 			(hide yes)
@@
 	)
 	(symbol
-		(lib_id "multi_fpga:C")
+		(lib_id "Device:C")
 		(at 111.76 58.42 0)
 		(unit 1)
@@
 		)
 		(property "Footprint" ""
+			(at 112.7252 62.23 0)
+			(hide yes)
+			(show_name no)
+			(do_not_autoplace no)
+			(effects
+				(font
+					(size 1.27 1.27)
+				)
+			)
+		)
+		(property "Datasheet" ""
 			(at 111.76 58.42 0)
 			(hide yes)
@@
 			)
 		)
-		(property "Datasheet" ""
+		(property "Description" "Unpolarized capacitor"
 			(at 111.76 58.42 0)
 			(hide yes)
@@
 			)
 		)
-		(property "Description" "100 nF decoupling capacitor, 0402"
-			(at 111.76 58.42 0)
-			(hide yes)
-			(show_name no)
-			(do_not_autoplace no)
-			(effects
-				(font
-					(size 1.27 1.27)
-				)
-			)
-		)
 		(pin "1"
 		)
@@
 	)
 	(symbol
-		(lib_id "multi_fpga:C")
+		(lib_id "Device:C")
 		(at 109.22 170.18 0)
 		(unit 1)
@@
 		)
 		(property "Footprint" ""
+			(at 110.1852 173.99 0)
+			(hide yes)
+			(show_name no)
+			(do_not_autoplace no)
+			(effects
+				(font
+					(size 1.27 1.27)
+				)
+			)
+		)
+		(property "Datasheet" ""
 			(at 109.22 170.18 0)
 			(hide yes)
@@
 			)
 		)
-		(property "Datasheet" ""
+		(property "Description" "Unpolarized capacitor"
 			(at 109.22 170.18 0)
 			(hide yes)
-			(show_name no)
-			(do_not_autoplace no)
-			(effects
-				(font
-					(size 1.27 1.27)
-				)
-			)
-		)
-		(property "Description" "100 nF decoupling capacitor, 0402"
-			(at 109.22 170.18 0)
-			(hide yes)

Commit message: Added stock footprints for C symbols.
Parts:
- C100, C101, C102, C103, C104, C105, C98, C99: footprint (none) -> Capacitor_SMD:C_0603_1608Metric
Changed lines of the file:
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@@
 			)
 		)
-		(property "Footprint" ""
+		(property "Footprint" "Capacitor_SMD:C_0603_1608Metric"
 			(at 107.6452 99.06 0)
 			(hide yes)
@@
 			)
 		)
-		(property "Footprint" ""
+		(property "Footprint" "Capacitor_SMD:C_0603_1608Metric"
 			(at 258.7752 215.9 0)
 			(hide yes)
@@
 			)
 		)
-		(property "Footprint" ""
+		(property "Footprint" "Capacitor_SMD:C_0603_1608Metric"
 			(at 108.9152 214.63 0)
 			(hide yes)
@@
 			)
 		)
-		(property "Footprint" ""
+		(property "Footprint" "Capacitor_SMD:C_0603_1608Metric"
 			(at 262.5852 62.23 0)
 			(hide yes)
@@
 			)
 		)
-		(property "Footprint" ""
+		(property "Footprint" "Capacitor_SMD:C_0603_1608Metric"
 			(at 257.5052 99.06 0)
 			(hide yes)
@@
 			)
 		)
-		(property "Footprint" ""
+		(property "Footprint" "Capacitor_SMD:C_0603_1608Metric"
 			(at 261.3152 175.26 0)
 			(hide yes)
@@
 			)
 		)
-		(property "Footprint" ""
+		(property "Footprint" "Capacitor_SMD:C_0603_1608Metric"
 			(at 112.7252 62.23 0)
 			(hide yes)
@@
 			)
 		)
-		(property "Footprint" ""
+		(property "Footprint" "Capacitor_SMD:C_0603_1608Metric"
 			(at 110.1852 173.99 0)
 			(hide yes)
