File: pcb/multi_fpga/arm_11.kicad_sch (KiCad schematic)
At the start: 16 parts, among them U89 IM72D128V01XTMA1, U90 IM72D128V01XTMA1, U91 IM72D128V01XTMA1, U92 IM72D128V01XTMA1, U93 IM72D128V01XTMA1, U94 IM72D128V01XTMA1, U95 IM72D128V01XTMA1, U96 IM72D128V01XTMA1

Commit message: Global fix of res defs.
Parts:
- renumbered C92 to C106, C90 to C107, C94 to C108, C93 to C109, C96 to C110, C91 to C111, C89 to C112, C95 to C113, U94 to U89, U89 to U90, U93 to U91, U90 to U92, U95 to U93, U91 to U94, U92 to U95

Commit message: Changed to use generic cap symbols and footprints.
Parts:
- C106, C107, C108, C109, C110, C111, C112, C113: symbol multi_fpga:C -> Device:C
Changed lines of the file:
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@@
 	)
 	(symbol
-		(lib_id "multi_fpga:C")
+		(lib_id "Device:C")
 		(at 107.95 210.82 0)
 		(unit 1)
@@
 		)
 		(property "Footprint" ""
-			(at 107.95 210.82 0)
+			(at 108.9152 214.63 0)
 			(hide yes)
 			(show_name no)
@@
 			)
 		)
-		(property "Description" "100 nF decoupling capacitor, 0402"
+		(property "Description" "Unpolarized capacitor"
 			(at 107.95 210.82 0)
 			(hide yes)
@@
 	)
 	(symbol
-		(lib_id "multi_fpga:C")
+		(lib_id "Device:C")
 		(at 106.68 95.25 0)
 		(unit 1)
@@
 		)
 		(property "Footprint" ""
-			(at 106.68 95.25 0)
+			(at 107.6452 99.06 0)
 			(hide yes)
 			(show_name no)
@@
 			)
 		)
-		(property "Description" "100 nF decoupling capacitor, 0402"
+		(property "Description" "Unpolarized capacitor"
 			(at 106.68 95.25 0)
 			(hide yes)
@@
 	)
 	(symbol
-		(lib_id "multi_fpga:C")
+		(lib_id "Device:C")
 		(at 261.62 58.42 0)
 		(unit 1)
@@
 		)
 		(property "Footprint" ""
-			(at 261.62 58.42 0)
+			(at 262.5852 62.23 0)
 			(hide yes)
 			(show_name no)
@@
 			)
 		)
-		(property "Description" "100 nF decoupling capacitor, 0402"
+		(property "Description" "Unpolarized capacitor"
 			(at 261.62 58.42 0)
 			(hide yes)
@@
 	)
 	(symbol
-		(lib_id "multi_fpga:C")
+		(lib_id "Device:C")
 		(at 109.22 170.18 0)
 		(unit 1)
@@
 		)
 		(property "Footprint" ""
-			(at 109.22 170.18 0)
+			(at 110.1852 173.99 0)
 			(hide yes)
 			(show_name no)
@@
 			)
 		)
-		(property "Description" "100 nF decoupling capacitor, 0402"
+		(property "Description" "Unpolarized capacitor"
 			(at 109.22 170.18 0)
 			(hide yes)
@@
 	)
 	(symbol
-		(lib_id "multi_fpga:C")
+		(lib_id "Device:C")
 		(at 256.54 95.25 0)
 		(unit 1)
@@
 		)
 		(property "Footprint" ""
-			(at 256.54 95.25 0)
+			(at 257.5052 99.06 0)
 			(hide yes)
 			(show_name no)
@@
 			)
 		)
-		(property "Description" "100 nF decoupling capacitor, 0402"
+		(property "Description" "Unpolarized capacitor"
 			(at 256.54 95.25 0)
 			(hide yes)
@@
 	)
 	(symbol
-		(lib_id "multi_fpga:C")
+		(lib_id "Device:C")
 		(at 111.76 58.42 0)
 		(unit 1)
@@
 		)
 		(property "Footprint" ""
-			(at 111.76 58.42 0)
+			(at 112.7252 62.23 0)
 			(hide yes)
 			(show_name no)
@@
 			)
 		)
-		(property "Description" "100 nF decoupling capacitor, 0402"
+		(property "Description" "Unpolarized capacitor"
 			(at 111.76 58.42 0)
 			(hide yes)
@@
 	)
 	(symbol
-		(lib_id "multi_fpga:C")
+		(lib_id "Device:C")
 		(at 257.81 212.09 0)
 		(unit 1)
@@
 		)
 		(property "Footprint" ""
-			(at 257.81 212.09 0)
+			(at 258.7752 215.9 0)
 			(hide yes)
 			(show_name no)
@@
 			)
 		)
-		(property "Description" "100 nF decoupling capacitor, 0402"
+		(property "Description" "Unpolarized capacitor"
 			(at 257.81 212.09 0)
 			(hide yes)
@@
 	)
 	(symbol
-		(lib_id "multi_fpga:C")
+		(lib_id "Device:C")
 		(at 260.35 171.45 0)
 		(unit 1)
@@
 		)
 		(property "Footprint" ""
-			(at 260.35 171.45 0)
+			(at 261.3152 175.26 0)
 			(hide yes)
 			(show_name no)
@@
 			)
 		)
-		(property "Description" "100 nF decoupling capacitor, 0402"
+		(property "Description" "Unpolarized capacitor"
 			(at 260.35 171.45 0)
 			(hide yes)

Commit message: Added stock footprints for C symbols.
Parts:
- C106, C107, C108, C109, C110, C111, C112, C113: footprint (none) -> Capacitor_SMD:C_0603_1608Metric
Changed lines of the file:
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@@
 			)
 		)
-		(property "Footprint" ""
+		(property "Footprint" "Capacitor_SMD:C_0603_1608Metric"
 			(at 108.9152 214.63 0)
 			(hide yes)
@@
 			)
 		)
-		(property "Footprint" ""
+		(property "Footprint" "Capacitor_SMD:C_0603_1608Metric"
 			(at 107.6452 99.06 0)
 			(hide yes)
@@
 			)
 		)
-		(property "Footprint" ""
+		(property "Footprint" "Capacitor_SMD:C_0603_1608Metric"
 			(at 262.5852 62.23 0)
 			(hide yes)
@@
 			)
 		)
-		(property "Footprint" ""
+		(property "Footprint" "Capacitor_SMD:C_0603_1608Metric"
 			(at 110.1852 173.99 0)
 			(hide yes)
@@
 			)
 		)
-		(property "Footprint" ""
+		(property "Footprint" "Capacitor_SMD:C_0603_1608Metric"
 			(at 257.5052 99.06 0)
 			(hide yes)
@@
 			)
 		)
-		(property "Footprint" ""
+		(property "Footprint" "Capacitor_SMD:C_0603_1608Metric"
 			(at 112.7252 62.23 0)
 			(hide yes)
@@
 			)
 		)
-		(property "Footprint" ""
+		(property "Footprint" "Capacitor_SMD:C_0603_1608Metric"
 			(at 258.7752 215.9 0)
 			(hide yes)
@@
 			)
 		)
-		(property "Footprint" ""
+		(property "Footprint" "Capacitor_SMD:C_0603_1608Metric"
 			(at 261.3152 175.26 0)
 			(hide yes)
