File: pcb/single_fpga/power_clock.kicad_sch (KiCad schematic)
At the start: 18 parts, among them J13 Main Power Input, U111 TLV62569DBV, U98 CDCLVC1112PW, Y1 ECS-TXO-5032

Commit message: Fixed buck converter wiring.
Connections:
- net GND: now also R4.1; no longer R3.2, R4.2
- net at U111.5 (FB): now also R3.2, R4.2; no longer R4.1
Other:
- moved on the sheet: C2, L1, R3, R4

Commit message: Fixed typo in signal name.
Connections:
- net ARM_11_CLK: no longer U98.14 (Y10)
- new net ARM_10_CLK: U98.14 (Y10)
Changed lines of the file:
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@@
 		)
 	)
-	(global_label "ARM_11_CLK"
+	(global_label "ARM_10_CLK"
 		(shape output)
 		(at 262.89 132.08 0)

Commit message: Fixed symbol library references.
Parts:
- C1: footprint 4ms_Capacitor:C_1206 -> PCM_4ms_Capacitor:C_1206
- U98: footprint PW24 -> CDCLVC1112:PW24
Changed lines of the file:
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@@
 			)
 		)
-		(property "Footprint" "4ms_Capacitor:C_1206"
+		(property "Footprint" "PCM_4ms_Capacitor:C_1206"
 			(at 55.88 120.65 0)
 			(hide yes)
@@
 			)
 		)
-		(property "Footprint" "PW24"
+		(property "Footprint" "CDCLVC1112:PW24"
 			(at 189.23 106.68 0)
 			(hide yes)
