File: pcb/single_fpga/mic_arm_00.kicad_sch (KiCad schematic)
At the start: 18 parts, among them U1 IM72D128V01XTMA1, U2 IM72D128V01XTMA1, U3 IM72D128V01XTMA1, U4 IM72D128V01XTMA1, U5 IM72D128V01XTMA1, U6 IM72D128V01XTMA1, U7 IM72D128V01XTMA1, U8 IM72D128V01XTMA1, U99 CDCLVC1108PW

Commit message: Fixed symbol library references.
Parts:
- U99: footprint PW0016A_N -> CDCLVC1108:PW0016A_N
Changed lines of the file:
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@@
 			)
 		)
-		(property "Footprint" "PW0016A_N"
+		(property "Footprint" "CDCLVC1108:PW0016A_N"
 			(at 229.87 95.25 0)
 			(hide yes)

Commit message: Fixed.
Other:
- moved on the sheet: C19, C22, U3, U4

Commit message: Fixed footprints. Added missing mic. Relinked placed footprints.
Parts:
- U1, U2, U3, U4, U5, U6, U7, U8: footprint (none) -> IM72D128:IFX-PG-LLGA-5-4
Changed lines of the file:
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@@
 			)
 		)
-		(property "Footprint" ""
+		(property "Footprint" "IM72D128:IFX-PG-LLGA-5-4"
 			(at 58.42 157.48 0)
 			(hide yes)
@@
 			)
 		)
-		(property "Footprint" ""
+		(property "Footprint" "IM72D128:IFX-PG-LLGA-5-4"
 			(at 135.89 160.02 0)
 			(hide yes)
@@
 			)
 		)
-		(property "Footprint" ""
+		(property "Footprint" "IM72D128:IFX-PG-LLGA-5-4"
 			(at 59.69 83.82 0)
 			(hide yes)
@@
 			)
 		)
-		(property "Footprint" ""
+		(property "Footprint" "IM72D128:IFX-PG-LLGA-5-4"
 			(at 58.42 118.11 0)
 			(hide yes)
@@
 			)
 		)
-		(property "Footprint" ""
+		(property "Footprint" "IM72D128:IFX-PG-LLGA-5-4"
 			(at 59.69 44.45 0)
 			(hide yes)
@@
 			)
 		)
-		(property "Footprint" ""
+		(property "Footprint" "IM72D128:IFX-PG-LLGA-5-4"
 			(at 135.89 83.82 0)
 			(hide yes)
@@
 			)
 		)
-		(property "Footprint" ""
+		(property "Footprint" "IM72D128:IFX-PG-LLGA-5-4"
 			(at 135.89 44.45 0)
 			(hide yes)
@@
 			)
 		)
-		(property "Footprint" ""
+		(property "Footprint" "IM72D128:IFX-PG-LLGA-5-4"
 			(at 135.89 120.65 0)
 			(hide yes)

Commit message: Updated all refdes's.
Parts:
- removed C18, C19, C20, C21, C22, C23, C24, C25: 100nF, Capacitor_SMD:C_0603_1608Metric, symbol Device:C
- removed R5: 10k, PCM_SparkFun-Resistor:R_0603_1608Metric, symbol PCM_SparkFun-Resistor:10k_0603
- removed U99: CDCLVC1108PW, CDCLVC1108:PW0016A_N, symbol CDCLVC1108:CDCLVC1108PW
- added C1, C2, C3, C4, C5, C6, C7, C8: 100nF, Capacitor_SMD:C_0603_1608Metric, symbol Device:C
- added R1: 10k, PCM_SparkFun-Resistor:R_0603_1608Metric, symbol PCM_SparkFun-Resistor:10k_0603
- added U9: CDCLVC1108PW, CDCLVC1108:PW0016A_N, symbol CDCLVC1108:CDCLVC1108PW
Connections:
- net ARM_00_CLK: now also U9.1 (CLKIN)
- net CLK_3V3: now also R1.2, U9.10 (VDD), U9.14 (VDD), U9.5 (VDD)
- net DATA_00: now also U3.1 (DATA), U4.1 (DATA); no longer U1.1 (DATA), U2.1 (DATA)
- net DATA_01: now also U1.1 (DATA), U2.1 (DATA); no longer U3.1 (DATA), U4.1 (DATA)
- net GND: now also C1.2, C2.2, C3.2, C4.2, C5.2, C6.2, C7.2, C8.2, U9.12 (GND), U9.4 (GND), U9.7 (GND)
- net MIC_3V3: now also C1.1, C2.1, C3.1, C4.1, C5.1, C6.1, C7.1, C8.1
- net MIC_CLK_00: now also U3.3 (CLK), U9.3 (Y0); no longer U1.3 (CLK)
- net MIC_CLK_01: now also U4.3 (CLK), U9.16 (Y1); no longer U2.3 (CLK)
- net MIC_CLK_02: now also U1.3 (CLK), U9.13 (Y2); no longer U3.3 (CLK)
- net MIC_CLK_03: now also U2.3 (CLK), U9.15 (Y3); no longer U4.3 (CLK)
- net MIC_CLK_04: now also U9.6 (Y4)
- net MIC_CLK_05: now also U9.11 (Y5)
- net MIC_CLK_06: now also U9.8 (Y6)
- net MIC_CLK_07: now also U9.9 (Y7)
- new net: R1.1, U9.2 (1G)

Commit message: Fixed res defs. New mic_array PCB layout.
Connections:
- net MIC_CLK_00: now also U1.3 (CLK); no longer U3.3 (CLK)
- net MIC_CLK_01: now also U2.3 (CLK); no longer U4.3 (CLK)
- net MIC_CLK_02: now also U3.3 (CLK); no longer U1.3 (CLK)
- net MIC_CLK_03: now also U4.3 (CLK); no longer U2.3 (CLK)
Other:
- moved on the sheet: C1, C2, C3, C4, U1, U2, U3, U4
