File: pcb/single_fpga/mic_array.kicad_pcb (KiCad board)
At the start: 2 copper layers, 320 x 320 mm, 220 parts, among them J1 AXK680337YG, J2 AXK680337YG, J3 AXK680337YG, J4 AXK680337YG, U1 Comment, U10 Comment, U100 PW0016A_N, U101 PW0016A_N, U102 PW0016A_N, U103 PW0016A_N, U104 PW0016A_N, U105 PW0016A_N, U106 PW0016A_N, U107 PW0016A_N, U108 PW0016A_N, U109 PW0016A_N, U11 Comment, U110 PW0016A_N, U12 Comment, U13 Comment, U14 Comment, U15 Comment, U16 Comment, U17 Comment, U18 Comment, U19 Comment, U2 Comment, U20 Comment, U21 Comment, U22 Comment, U23 Comment, U24 Comment, U25 Comment, U26 Comment, U27 Comment, U28 Comment, U29 Comment, U3 Comment, U30 Comment, U31 Comment, U32 Comment, U33 Comment, U34 Comment, U35 Comment, U36 Comment, U37 Comment, U38 Comment, U39 Comment, U4 Comment, U40 Comment, U41 Comment, U42 Comment, U43 Comment, U44 Comment, U45 Comment, U46 Comment, U47 Comment, U48 Comment, U49 Comment, U5 Comment, U50 Comment, U51 Comment, U52 Comment, U53 Comment, U54 Comment, U55 Comment, U56 Comment, U57 Comment, U58 Comment, U59 Comment, U6 Comment, U60 Comment, U61 Comment, U62 Comment, U63 Comment, U64 Comment, U65 Comment, U66 Comment, U67 Comment, U68 Comment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

Commit message: Fixed footprints. Added missing mic. Relinked placed footprints.
Parts:
- C100, C101, C102, C103, C104, C105, C106, C107, C108, C109, C110, C111, C112, C113, C18, C19, C20, C21, C22, C23, C24, C25, C26, C27, C28, C29, C30, C31, C32, C33, C34, C35, C36, C37, C38, C39, C40, C41, C42, C43, C44, C45, C46, C47, C48, C49, C50, C51, C52, C53, C54, C55, C56, C57, C58, C59, C60, C61, C62, C63, C64, C65, C66, C67, C68, C69, C70, C71, C72, C73, C74, C75, C76, C77, C78, C79, C80, C81, C82, C83, C84, C85, C86, C87, C88, C89, C90, C91, C92, C93, C94, C95, C96, C97, C98, C99: footprint C_0603_1608Metric -> Capacitor_SMD:C_0603_1608Metric
- U1, U10, U11, U12, U13, U14, U15, U16, U17, U18, U19, U2, U20, U21, U22, U23, U24, U25, U26, U27, U28, U29, U3, U30, U31, U32, U33, U34, U35, U36, U37, U38, U39, U4, U40, U41, U42, U43, U44, U45, U46, U47, U48, U49, U5, U50, U51, U52, U53, U54, U55, U56, U57, U58, U59, U6, U60, U61, U62, U63, U64, U65, U66, U67, U68, U69, U7, U70, U71, U72, U73, U74, U75, U76, U77, U78, U79, U8, U80, U81, U82, U83, U84, U85, U86, U87, U88, U89, U9, U90, U91, U92, U93, U94, U95, U96: footprint IFX-PG-LLGA-5-4 -> IM72D128:IFX-PG-LLGA-5-4

Commit message: Changed inter-board connectors (J1 and J2) to be taller.
Parts:
- added C114: 1uF, Capacitor_SMD:C_1206_3216Metric, F.Cu at (59.4, 96.4)
- added C115: 1uF, Capacitor_SMD:C_1206_3216Metric, F.Cu at (59.4, 99.7)
- added C15: .1uF, Capacitor_SMD:C_0603_1608Metric, F.Cu at (58.6, 102.7)
- added C16: 1uF, Capacitor_SMD:C_1206_3216Metric, F.Cu at (59.4, 89.7)
- added C17: 1uF, Capacitor_SMD:C_1206_3216Metric, F.Cu at (59.4, 93.0)
- added R10: 10k, PCM_SparkFun-Resistor:R_0603_1608Metric, F.Cu at (100.9, 50.3)
- added R11: 10k, PCM_SparkFun-Resistor:R_0603_1608Metric, F.Cu at (43.8, 79.8)
- added R12: 10k, PCM_SparkFun-Resistor:R_0603_1608Metric, F.Cu at (15.2, 50.3)
- added R13: 10k, PCM_SparkFun-Resistor:R_0603_1608Metric, F.Cu at (43.8, 20.8)
- added R14: 10k, PCM_SparkFun-Resistor:R_0603_1608Metric, F.Cu at (43.8, 50.3)
- added R15: 10k, PCM_SparkFun-Resistor:R_0603_1608Metric, F.Cu at (15.2, 20.8)
- added R16: 10k, PCM_SparkFun-Resistor:R_0603_1608Metric, F.Cu at (72.3, 20.8)
- added R2: 10k, PCM_SparkFun-Resistor:R_0603_1608Metric, F.Cu at (58.6, 105.2)
- added R5: 10k, PCM_SparkFun-Resistor:R_0603_1608Metric, F.Cu at (100.9, 20.8)
- added R6: 10k, PCM_SparkFun-Resistor:R_0603_1608Metric, F.Cu at (15.2, 79.8)
- added R7: 10k, PCM_SparkFun-Resistor:R_0603_1608Metric, F.Cu at (100.9, 79.8)
- added R8: 10k, PCM_SparkFun-Resistor:R_0603_1608Metric, F.Cu at (72.3, 50.3)
- added R9: 10k, PCM_SparkFun-Resistor:R_0603_1608Metric, F.Cu at (72.3, 79.8)
- added U98: CDCLVC1112PW, CDCLVC1112:PW24, F.Cu at (66.9, 92.8)
- added VR5: MCP1700T-3302E/TT, Package_TO_SOT_SMD:SOT-23, F.Cu at (64.7, 99.8)
- added VR6: MCP1700T-3302E/TT, Package_TO_SOT_SMD:SOT-23, F.Cu at (64.7, 104.2)
- added Y1: ECS-TXO-5032, multi_fpga:ECS-TXO-5032-122.8-TR, F.Cu at (71.2, 100.1)
- J1, J2: value AXK680337YG -> AXK6S80347YG; footprint AXK680337YG -> AXK6S80347YG:CONN80_AXK6S80347YG_PAN

Commit message: Fixed problems caused by saving from top.kicad_pro.
Parts:
- removed HAC1, HAC2, HAC3, HAC4: MountingHole_2.7mm_M2.5, MountingHole_2.7mm_M2.5
- removed J2: AXK6S80347YG, AXK6S80347YG:CONN80_AXK6S80347YG_PAN
- removed J3, J4: AXK680337YG, AXK680337YG
- removed R10, R11, R12, R13, R14, R15, R16, R5, R6, R7, R8, R9: 10k, PCM_SparkFun-Resistor:R_0603_1608Metric
- J1: moved to F.Cu
- moved J1 284.1 mm to (269.3, 191.5), turned to 0 degrees
- moved C115 245.3 mm to (285.0, 196.0)
- moved VR5 240.8 mm to (283.9, 199.5), turned to 180 degrees
- moved C17 239.8 mm to (274.5, 199.0)
- moved U98 237.3 mm to (268.5, 218.0)
- moved Y1 235.6 mm to (279.0, 211.3)
- moved C114 231.9 mm to (260.5, 212.0)
- moved C16 231.0 mm to (263.0, 199.0)
- moved C15 216.8 mm to (254.3, 196.0)
- moved VR6 212.5 mm to (254.4, 200.0)
- moved R2 210.0 mm to (247.0, 198.0)

Commit message: Fixed ref des's to match schematics.
Parts:
- removed C102, C103, C104, C105, C106, C107, C108, C109, C110, C111, C112, C113: C_0603_1608Metric, Capacitor_SMD:C_0603_1608Metric
- removed C114, C115: 1uF, Capacitor_SMD:C_1206_3216Metric
- removed U109: PW0016A_N, CDCLVC1108:PW0016A_N
- removed VR5, VR6: MCP1700T-3302E/TT, Package_TO_SOT_SMD:SOT-23
- added C1: 100nF, C_0603_1608Metric, F.Cu at (293.4, 202.4)
- added C10: 100nF, C_0603_1608Metric, F.Cu at (307.0, 249.3)
- added C11: 100nF, C_0603_1608Metric, F.Cu at (311.7, 267.9)
- added C12: 100nF, C_0603_1608Metric, F.Cu at (314.8, 287.0)
- added C13: 100nF, C_0603_1608Metric, F.Cu at (316.3, 306.1)
- added C14: 100nF, C_0603_1608Metric, F.Cu at (316.7, 325.4)
- added C2: 100nF, C_0603_1608Metric, F.Cu at (310.2, 211.7)
- added C3: 100nF, C_0603_1608Metric, F.Cu at (325.2, 223.7)
- added C4: 100nF, C_0603_1608Metric, F.Cu at (338.7, 237.5)
- added C5: 100nF, C_0603_1608Metric, F.Cu at (350.8, 252.4)
- added C6: 100nF, C_0603_1608Metric, F.Cu at (361.8, 268.3)
- added C7: 100nF, C_0603_1608Metric, F.Cu at (371.7, 284.8)
- added C8: 100nF, C_0603_1608Metric, F.Cu at (380.8, 301.8)
- added C9: 100nF, C_0603_1608Metric, F.Cu at (300.0, 231.4)
- added R1: 10k, R_0603_1608Metric, F.Cu at (298.9, 205.4)
- added R10: 10k, R_0603_1608Metric, F.Cu at (377.6, 157.4)
- added R11: 10k, R_0603_1608Metric, F.Cu at (333.8, 195.4)
- added R12: 10k, R_0603_1608Metric, F.Cu at (318.7, 280.4)
- added R13: 10k, R_0603_1608Metric, F.Cu at (269.2, 210.0)
- added R3: 10k, R_0603_1608Metric, F.Cu at (244.0, 352.4)
- added R4: 10k, R_0603_1608Metric, F.Cu at (174.5, 317.7)
- added R5: 10k, R_0603_1608Metric, F.Cu at (177.5, 203.3)
- added R6: 10k, R_0603_1608Metric, F.Cu at (143.2, 185.7)
- added R7: 10k, R_0603_1608Metric, F.Cu at (225.5, 82.4)
- added R8: 10k, R_0603_1608Metric, F.Cu at (263.9, 145.5)
- added R9: 10k, R_0603_1608Metric, F.Cu at (308.9, 135.1)
- added U97: IM72D128V01XTMA1, IFX-PG-LLGA-5-4, F.Cu at (432.2, 245.4)
- added VR1: MCP1700T-3302E/TT, SOT-23, F.Cu at (283.9, 199.5)
- added VR2: MCP1700T-3302E/TT, SOT-23, F.Cu at (254.4, 200.0)
- J1: footprint AXK6S80347YG:CONN80_AXK6S80347YG_PAN -> CONN80_AXK6S80347YG_PAN

Commit message: Fixed res defs. New mic_array PCB layout.
Parts:
- C100, C101, C98, C99: value C_0603_1608Metric -> 1uF; footprint Capacitor_SMD:C_0603_1608Metric -> C_1206_3216Metric
- C15: value .1uF -> 100nF; footprint Capacitor_SMD:C_0603_1608Metric -> C_0603_1608Metric
- C16, C17: value 1uF -> 100nF; footprint Capacitor_SMD:C_1206_3216Metric -> C_0603_1608Metric
- C18, C19, C20, C21, C22, C23, C24, C25, C26, C27, C28, C29, C30, C31, C32, C33, C34, C35, C36, C37, C38, C39, C40, C41, C42, C43, C44, C45, C46, C47, C48, C49, C50, C51, C52, C53, C54, C55, C56, C57, C58, C59, C60, C61, C62, C63, C64, C65, C66, C67, C68, C69, C70, C71, C72, C73, C74, C75, C76, C77, C78, C79, C80, C81, C82, C83, C84, C85, C86, C87, C88, C89, C90, C91, C92, C93, C94, C95, C96: value C_0603_1608Metric -> 100nF; footprint Capacitor_SMD:C_0603_1608Metric -> C_0603_1608Metric
- C97: value C_0603_1608Metric -> .1uF; footprint Capacitor_SMD:C_0603_1608Metric -> C_0603_1608Metric
- R2: footprint PCM_SparkFun-Resistor:R_0603_1608Metric -> R_0603_1608Metric
- U1, U10, U11, U12, U13, U14, U15, U16, U17, U19, U2, U20, U21, U22, U23, U24, U25, U26, U28, U29, U3, U30, U31, U32, U33, U34, U35, U37, U38, U39, U4, U40, U41, U42, U43, U44, U46, U47, U48, U49, U5, U50, U51, U52, U53, U55, U56, U57, U58, U59, U6, U60, U61, U62, U64, U65, U66, U67, U68, U69, U7, U70, U71, U73, U74, U75, U76, U77, U78, U79, U8, U80, U82, U83, U84, U85, U86, U87, U88, U89, U91, U92, U93, U94, U95, U96: value Comment -> IM72D128V01XTMA1; footprint IM72D128:IFX-PG-LLGA-5-4 -> IFX-PG-LLGA-5-4
- U100, U101, U102, U103, U104, U105, U106, U107: value PW0016A_N -> IM72D128V01XTMA1; footprint CDCLVC1108:PW0016A_N -> IFX-PG-LLGA-5-4
- U108, U99: value PW0016A_N -> CDCLVC1108PW; footprint CDCLVC1108:PW0016A_N -> PW0016A_N
- U110: value PW0016A_N -> CDCLVC1112PW; footprint CDCLVC1108:PW0016A_N -> PW24
- U18, U27, U36, U45, U54, U63, U72, U81, U9, U90: value Comment -> CDCLVC1108PW; footprint IM72D128:IFX-PG-LLGA-5-4 -> PW0016A_N
- U98: value CDCLVC1112PW -> IM72D128V01XTMA1; footprint CDCLVC1112:PW24 -> IFX-PG-LLGA-5-4
- Y1: footprint multi_fpga:ECS-TXO-5032-122.8-TR -> ECS-TXO-5032-122.8-TR
- moved U106 199.4 mm to (399.5, 225.0)
- moved U105 197.4 mm to (382.7, 215.7)
- moved U107 189.1 mm to (415.9, 235.2)
- moved U104 183.8 mm to (365.3, 207.5)
- moved R2 163.9 mm to (301.3, 352.7)
- moved U103 161.3 mm to (347.3, 200.6)
- moved U98 154.8 mm to (411.1, 157.7)
- moved U108 154.8 mm to (413.9, 245.0)
- moved C94 148.6 mm to (415.4, 232.3)
- moved C22 148.6 mm to (238.5, 349.4)
- moved C86 148.5 mm to (410.6, 154.8)
- moved C30 148.4 mm to (169.0, 314.8)
- moved C78 148.3 mm to (367.7, 90.0)
- moved C38 148.3 mm to (126.1, 250.1)
- moved C70 148.2 mm to (298.2, 55.4)
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Connections:
- C15 pad 1: CLK_3V3 -> (no net)
- C15 pad 2: GND -> (no net)
- C16 pad 1: +3V6 -> (no net)
- C16 pad 2: GND -> (no net)
- C17 pad 1: MIC_3V3 -> (no net)
- C17 pad 2: GND -> (no net)
- R2 pad 1: Net-(U98-1G) -> (no net)
- R2 pad 2: CLK_3V3 -> (no net)
- U98 pad 1: TCXO_CLK -> (no net)
- U98 pad 2: Net-(U98-1G) -> (no net)
- U98 pad 3: ARM_00_CLK -> (no net)
- U98 pad 4: GND -> (no net)
- U98 pad 5: CLK_3V3 -> (no net)
- Y1 pad 1: unconnected-(Y1-VCONT-Pad1) -> (no net)
- Y1 pad 2: GND -> (no net)
- Y1 pad 3: TCXO_CLK -> (no net)
- Y1 pad 4: CLK_3V3 -> (no net)

Commit message: Moved caps and mic ref des labels.
Parts:
- moved U110 88.9 mm to (268.4, 217.6)
- moved C100 8.93 mm to (307.5, 159.1)
- moved C101 6.00 mm to (333.9, 152.8)
- moved C97 6.00 mm to (367.7, 83.7)
- moved C98 6.00 mm to (280.9, 174.5)
- moved C99 6.00 mm to (297.3, 164.5)

Commit message: Moved mic caps a little more. Moved per-arm clock drivers to mid-arm.
Parts:
- moved U9 66.3 mm to (341.3, 254.9)
- moved U36 66.3 mm to (219.3, 277.8)
- moved U63 66.3 mm to (196.4, 155.8)
- moved U90 66.3 mm to (318.4, 132.9)
- moved U108 66.3 mm to (356.4, 212.0)
- moved U27 66.3 mm to (262.2, 292.9)
- moved U81 66.3 mm to (275.5, 117.8)
- moved U54 66.3 mm to (181.3, 198.7)
- moved U18 66.3 mm to (306.9, 284.5)
- moved U99 66.3 mm to (348.0, 167.4)
- moved U45 66.3 mm to (189.7, 243.4)
- moved U72 66.3 mm to (230.9, 126.2)
- moved C100 3.00 mm to (304.6, 160.0)
- moved C101 3.00 mm to (333.9, 149.8)
- moved C98 3.00 mm to (280.9, 171.5)
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Changed lines of the file:
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@@
 	(footprint "C_1206_3216Metric"
 		(layer "F.Cu")
-		(at 307.5 159.09)
+		(at 304.65 160.03)
 		(descr "Capacitor SMD 1206 (3216 Metric), square (rectangular) end terminal, IPC-7351 nominal, (Body size source: IPC-SM-782 page 76, https://www.pcb-3d.com/wordpress/wp-content/uploads/ipc-sm-782a_amendment_1_and_2.pdf)")
 		(tags "capacitor")
@@
 	(footprint "PW0016A_N"
 		(layer "F.Cu")
-		(at 230.693201 59.956336)
+		(at 230.859694 126.22346)
 		(tags "CDCLVC1108PW ")
 		(property "Reference" "U72"
@@
 	(footprint "PW0016A_N"
 		(layer "F.Cu")
-		(at 123.456335 243.532629)
+		(at 189.723459 243.366136)
 		(tags "CDCLVC1108PW ")
 		(property "Reference" "U45"
@@
 	(footprint "PW0016A_N"
 		(layer "F.Cu")
-		(at 123.852234 165.715584)
+		(at 181.3246 198.704907)
 		(tags "CDCLVC1108PW ")
 		(property "Reference" "U54"
@@
 	(footprint "PW0016A_N"
 		(layer "F.Cu")
-		(at 308.510246 60.352235)
+		(at 275.520923 117.824601)
 		(tags "CDCLVC1108PW ")
 		(property "Reference" "U81"
@@
 	(footprint "C_0603_1608Metric"
 		(layer "F.Cu")
-		(at 367.721716 83.730416)
+		(at 367.721716 82.23)
 		(descr "Capacitor SMD 0603 (1608 Metric), square (rectangular) end terminal, IPC-7351 nominal, (Body size source: IPC-SM-782 page 76, https://www.pcb-3d.com/wordpress/wp-content/uploads/ipc-sm-782a_amendment_1_and_2.pdf)")
 		(tags "capacitor")
@@
 	(footprint "C_1206_3216Metric"
 		(layer "F.Cu")
-		(at 333.899116 152.756316)
+		(at 333.899116 149.756316)
 		(descr "Capacitor SMD 1206 (3216 Metric), square (rectangular) end terminal, IPC-7351 nominal, (Body size source: IPC-SM-782 page 76, https://www.pcb-3d.com/wordpress/wp-content/uploads/ipc-sm-782a_amendment_1_and_2.pdf)")
 		(tags "capacitor")
@@
 	(footprint "PW0016A_N"
 		(layer "F.Cu")
-		(at 414.269494 167.193202)
+		(at 348.00237 167.359695)
 		(tags "CDCLVC1108PW ")
 		(property "Reference" "U99"
@@
 	(footprint "PW0016A_N"
 		(layer "F.Cu")
-		(at 413.873595 245.010247)
+		(at 356.401229 212.020924)
 		(tags "CDCLVC1108PW ")
 		(property "Reference" "U108"
@@
 	(footprint "PW0016A_N"
 		(layer "F.Cu")
-		(at 162.02195 311.122164)
+		(at 219.327768 277.844363)
 		(tags "CDCLVC1108PW ")
 		(property "Reference" "U36"
@@
 	(footprint "PW0016A_N"
 		(layer "F.Cu")
-		(at 375.703879 99.603667)
+		(at 318.398061 132.881468)
 		(tags "CDCLVC1108PW ")
 		(property "Reference" "U90"
@@
 	(footprint "PW0016A_N"
 		(layer "F.Cu")
-		(at 229.215583 350.373596)
+		(at 262.204906 292.90123)
 		(tags "CDCLVC1108PW ")
 		(property "Reference" "U27"
@@
 	(footprint "PW0016A_N"
 		(layer "F.Cu")
-		(at 307.032628 350.769495)
+		(at 306.866135 284.502371)
 		(tags "CDCLVC1108PW ")
 		(property "Reference" "U18"
@@
 	(footprint "PW0016A_N"
 		(layer "F.Cu")
-		(at 163.103666 98.521951)
+		(at 196.381467 155.827769)
 		(tags "CDCLVC1108PW ")
 		(property "Reference" "U63"
@@
 	(footprint "C_1206_3216Metric"
 		(layer "F.Cu")
-		(at 280.872916 174.462316)
+		(at 280.872916 171.462316)
 		(descr "Capacitor SMD 1206 (3216 Metric), square (rectangular) end terminal, IPC-7351 nominal, (Body size source: IPC-SM-782 page 76, https://www.pcb-3d.com/wordpress/wp-content/uploads/ipc-sm-782a_amendment_1_and_2.pdf)")
 		(tags "capacitor")
@@
 	(footprint "C_1206_3216Metric"
 		(layer "F.Cu")
-		(at 297.314216 164.503816)
+		(at 297.314216 161.503816)
 		(descr "Capacitor SMD 1206 (3216 Metric), square (rectangular) end terminal, IPC-7351 nominal, (Body size source: IPC-SM-782 page 76, https://www.pcb-3d.com/wordpress/wp-content/uploads/ipc-sm-782a_amendment_1_and_2.pdf)")
 		(tags "capacitor")
@@
 	(footprint "PW0016A_N"
 		(layer "F.Cu")
-		(at 374.622163 312.20388)
+		(at 341.344362 254.898062)
 		(tags "CDCLVC1108PW ")
 		(property "Reference" "U9"

Commit message: Cleaned up silk-screen overlaps. Moved clock driver resistors closer.
Parts:
- moved R12 62.2 mm to (356.6, 224.0)
- moved R3 62.2 mm to (250.2, 293.1)
- moved R6 62.2 mm to (181.1, 186.7)
- moved R9 62.2 mm to (287.5, 117.6)
- moved R4 62.2 mm to (208.8, 272.0)
- moved R7 62.2 mm to (202.2, 145.3)
- moved R1 62.2 mm to (335.5, 265.4)
- moved R10 62.2 mm to (328.9, 138.7)
- moved R11 62.2 mm to (354.2, 177.7)
- moved R5 62.2 mm to (183.6, 233.1)
- moved R8 62.2 mm to (241.2, 120.1)
- moved R2 62.2 mm to (296.6, 290.7)
- moved C17 1.50 mm to (281.0, 241.8)
- moved C60 1.50 mm to (229.5, 154.1)
- moved C84 1.50 mm to (315.0, 162.4)
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